File: SpeakerAdapter.sch (KiCad schematic (older format))
At the start: 51 parts

Commit message: Add JST-PH connector.
Parts:
- added J?: JST-PH, Connector_JST:JST_PH_B4B-PH-K_1x04_P2.00mm_Vertical, symbol Connector_Generic:Conn_01x04
Other:
- moved on the sheet: J?
Changed lines of the file:
@@
 EESchema Schematic File Version 4
-LIBS:navigation-board-cache
 EELAYER 26 0
 EELAYER END
@@
 L Connector:Screw_Terminal_01x04 J?
 U 1 1 5D7189D5
-P 4000 2700
-F 0 "J?" H 4079 2692 50  0000 L CNN
-F 1 "Terminal Block" H 4079 2601 50  0000 L CNN
-F 2 "TerminalBlock_4Ucon:TerminalBlock_4Ucon_1x04_P3.50mm_Horizontal" H 4000 2700 50  0001 C CNN
-F 3 "~" H 4000 2700 50  0001 C CNN
-F 4 "1776275-4" H 4000 2700 50  0001 C CNN "MPN"
-F 5 "TERM BLK 4POS SIDE ENT 3.5MM PCB" H 4000 2700 50  0001 C CNN "Description"
-F 6 "A98038-ND" H 4000 2700 50  0001 C CNN "Digi-Key_PN"
-	1    4000 2700
-	1    0    0    -1
-$EndComp
+P 7800 6000
+F 0 "J?" H 7879 5992 50  0000 L CNN
+F 1 "Terminal Block" H 7879 5901 50  0000 L CNN
+F 2 "TerminalBlock_4Ucon:TerminalBlock_4Ucon_1x04_P3.50mm_Horizontal" H 7800 6000 50  0001 C CNN
+F 3 "~" H 7800 6000 50  0001 C CNN
+F 4 "1776275-4" H 7800 6000 50  0001 C CNN "MPN"
+F 5 "TERM BLK 4POS SIDE ENT 3.5MM PCB" H 7800 6000 50  0001 C CNN "Description"
+F 6 "A98038-ND" H 7800 6000 50  0001 C CNN "Digi-Key_PN"
+	1    7800 6000
+	1    0    0    -1
+$EndComp
+$Comp
+L Connector_Generic:Conn_01x04 J?
+U 1 1 5D619CD2
+P 9100 6000
+F 0 "J?" H 9179 5992 50  0000 L CNN
+F 1 "JST-PH" H 9179 5901 50  0000 L CNN
+F 2 "Connector_JST:JST_PH_B4B-PH-K_1x04_P2.00mm_Vertical" H 9100 6000 50  0001 C CNN
+F 3 "http://www.jst-mfg.com/product/pdf/eng/ePH.pdf" H 9100 6000 50  0001 C CNN
+F 4 "B4B-PH-K-S(LF)(SN)" H 9100 6000 50  0001 C CNN "MPN"
+F 5 "CONN HEADER VERT 4POS 2MM" H 9100 6000 50  0001 C CNN "Description"
+F 6 "455-1706-ND" H 9100 6000 50  0001 C CNN "Digi-Key_PN"
+	1    9100 6000
+	1    0    0    -1
+$EndComp

Commit message: Remove unused palette items.
Parts:
- removed C?: 30pF, Capacitor_THT:C_Disc_D3.8mm_W2.6mm_P2.50mm, symbol Device:C
- removed C?: 0.01μF, Capacitor_THT:C_Disc_D12.5mm_W5.0mm_P7.50mm, symbol Device:C
- removed C?: 0.1μF, Capacitor_THT:C_Disc_D3.8mm_W2.6mm_P2.50mm, symbol Device:C
- removed C?: 0.22μF, Capacitor_THT:C_Disc_D7.5mm_W4.4mm_P5.00mm, symbol Device:C
- removed C?: 22pF, Capacitor_THT:C_Disc_D3.8mm_W2.6mm_P2.50mm, symbol Device:C
- removed C?: 1μF, Capacitor_THT:C_Disc_D3.8mm_W2.6mm_P2.50mm, symbol Device:C
- removed C?: 10μF, Capacitor_THT:C_Disc_D5.1mm_W3.2mm_P5.00mm, symbol Device:C
- removed D?: 1N4007, Diode_THT:D_DO-41_SOD81_P7.62mm_Horizontal, symbol Device:D_ALT
- removed D?: D_Bridge_+-AA, Diode_THT:Diode_Bridge_DIP-4_W7.62mm_P5.08mm, symbol Device:D_Bridge_+-AA
- removed J?: ISP6, local:IDC-Header_2x03_P2.54mm_Vertical, symbol avr-arduino:ISP6
- removed J?: 87180-062LF, digikey-footprints:Phone_Jack_87180-062LF, symbol dk_Modular-Connectors-Jacks:87180-062LF
- removed J?: Screw_Terminal_01x01, local:Screw_Terminal_M4_Keystone_7796, symbol Connector:Screw_Terminal_01x01
- removed J?: Barrel_Jack_MountingPin, Connector_BarrelJack:BarrelJack_CUI_PJ-063AH_Horizontal, symbol Connector:Barrel_Jack_MountingPin
- removed J?: USB_A, local:USB_A_Vertical, symbol Connector:USB_A
- removed J?: IDC 20, local:IDC-Header_2x10_P2.54mm_Vertical, symbol Connector_Generic:Conn_02x10_Odd_Even
- removed J?: IDC 16, symbol Connector_Generic:Conn_02x08_Odd_Even
- removed J?: 6 pin female, Connector_PinSocket_2.54mm:PinSocket_1x06_P2.54mm_Vertical, symbol Connector_Generic:Conn_01x06
- removed J?: 12 pin female, Connector_PinSocket_2.54mm:PinSocket_1x12_P2.54mm_Vertical, symbol Connector_Generic:Conn_01x12
- removed J?: 4 pin RA male, Connector_PinHeader_2.54mm:PinHeader_1x04_P2.54mm_Horizontal, symbol Connector_Generic:Conn_01x04
- removed J?: Grove Horizontal, local:NS-Tech_Grove_1x04_P2mm_Horizontal, symbol Connector_Generic:Conn_01x04
- removed J?: Grove Vertical, Connector:NS-Tech_Grove_1x04_P2mm_Vertical, symbol Connector_Generic:Conn_01x04
- removed K?: G5RL-U1A-E, local:Relay_SPST_Omron-G5RL-U1A-E, symbol local:G5RL-U1A-E
- removed K?: G5RL-K1-E, local:Relay_SPDT_Omron-G5RL-K1-E, symbol local:G5RL-K1-E
- removed LS?: Speaker, local:Speaker_CVS-1508, symbol Device:Speaker
- removed Q?: 2N4401, Package_TO_SOT_THT:TO-92_Inline_Wide, symbol Device:Q_NPN_EBC
- removed Q?: BS107, Package_TO_SOT_THT:TO-92_Inline, symbol Transistor_FET:BS107
- removed R?: 1K, Resistor_THT:R_Axial_DIN0207_L6.3mm_D2.5mm_P2.54mm_Vertical, symbol Device:R_US
- removed R?: 390, Resistor_THT:R_Axial_DIN0207_L6.3mm_D2.5mm_P2.54mm_Vertical, symbol Device:R_US
- removed R?: 15k, Resistor_THT:R_Axial_DIN0207_L6.3mm_D2.5mm_P2.54mm_Vertical, symbol Device:R_US
- removed R?: 18k, Resistor_THT:R_Axial_DIN0207_L6.3mm_D2.5mm_P2.54mm_Vertical, symbol Device:R_US
- removed R?: 200k, Resistor_THT:R_Axial_DIN0207_L6.3mm_D2.5mm_P2.54mm_Vertical, symbol Device:R_US
- removed R?: 470k, Resistor_THT:R_Axial_DIN0207_L6.3mm_D2.5mm_P2.54mm_Vertical, symbol Device:R_US
- removed R?: 10M, Resistor_THT:R_Axial_DIN0207_L6.3mm_D2.5mm_P2.54mm_Vertical, symbol Device:R_US
- removed R?: 270k, Resistor_THT:R_Axial_DIN0207_L6.3mm_D2.5mm_P2.54mm_Vertical, symbol Device:R_US
- removed R?: 20k, Resistor_THT:R_Axial_DIN0207_L6.3mm_D2.5mm_P2.54mm_Vertical, symbol Device:R_US
- removed R?: 10k, Resistor_THT:R_Axial_DIN0207_L6.3mm_D2.5mm_P2.54mm_Vertical, symbol Device:R_US
- removed SW?: Green, local:SW_PUSH_E-Switch_TL6215R, symbol Switch:SW_Push_LED
- removed SW?: Blue, local:SW_PUSH_E-Switch_TL6215R, symbol Switch:SW_Push_LED
- removed SW?: Red, local:SW_PUSH_E-Switch_TL6215R, symbol Switch:SW_Push_LED
- removed SW?: SW_Navigation, local:SW_Navigation_SKQUCAA010, symbol local:SW_Navigation
- removed U?: H11L1, Package_DIP:DIP-6_W7.62mm, symbol Isolator:H11L1
- removed U?: HT9032C, Package_DIP:DIP-16_W7.62mm_Socket, symbol local:HT9032C
- removed U?: AVR_28DIP_Arduino, Housings_DIP:DIP-28_W7.62mm, symbol avr-arduino:AVR_28DIP_Arduino
- removed U?: SN754410, Package_DIP:DIP-16_W7.62mm, symbol Driver_Motor:L293D
- removed U?: 74LVC245, symbol 74xx:74HC245
- removed U?: MCP1702-3302E_TO92, Package_TO_SOT_THT:TO-92_Inline, symbol Regulator_Linear:MCP1700-3302E_TO92
- removed U?: TSR_1-2433, Converter_DCDC:Converter_DCDC_TRACO_TSR-1_THT, symbol Regulator_Switching:TSR_1-2433
- removed U?: TSOP38238, digikey-footprints:IR_Receiver_TSOP38238, symbol dk_Optical-Sensors-Photo-Detectors-Remote-Receiver:TSOP38238
- removed Y?: 3.579545MHz, Crystal:Crystal_HC49-U_Vertical, symbol Device:Crystal
- removed Y?: 16MHz, Crystal:Crystal_HC49-U_Vertical, symbol Device:Crystal
Other:
- note removed: "+"

Commit message: Draw schematic.
Parts:
- gave numbers to parts that had none: 2
Connections:
- net at J2.1 (Pin_1): now also J1.1 (Pin_1)
- net at J2.2 (Pin_2): now also J1.2 (Pin_2)
- net at J2.3 (Pin_3): now also J1.3 (Pin_3)
- net at J2.4 (Pin_4): now also J1.4 (Pin_4)
Other:
- moved on the sheet: J1
Changed lines of the file:
@@
 $EndDescr
 $Comp
-L Connector:Screw_Terminal_01x04 J?
+L Connector:Screw_Terminal_01x04 J1
 U 1 1 5D7189D5
-P 7800 6000
-F 0 "J?" H 7879 5992 50  0000 L CNN
-F 1 "Terminal Block" H 7879 5901 50  0000 L CNN
-F 2 "TerminalBlock_4Ucon:TerminalBlock_4Ucon_1x04_P3.50mm_Horizontal" H 7800 6000 50  0001 C CNN
-F 3 "~" H 7800 6000 50  0001 C CNN
-F 4 "1776275-4" H 7800 6000 50  0001 C CNN "MPN"
-F 5 "TERM BLK 4POS SIDE ENT 3.5MM PCB" H 7800 6000 50  0001 C CNN "Description"
-F 6 "A98038-ND" H 7800 6000 50  0001 C CNN "Digi-Key_PN"
-	1    7800 6000
-	1    0    0    -1
+P 8200 6000
+F 0 "J1" H 8279 5992 50  0000 L CNN
+F 1 "Terminal Block" H 8279 5901 50  0000 L CNN
+F 2 "TerminalBlock_4Ucon:TerminalBlock_4Ucon_1x04_P3.50mm_Horizontal" H 8200 6000 50  0001 C CNN
+F 3 "~" H 8200 6000 50  0001 C CNN
+F 4 "1776275-4" H 8200 6000 50  0001 C CNN "MPN"
+F 5 "TERM BLK 4POS SIDE ENT 3.5MM PCB" H 8200 6000 50  0001 C CNN "Description"
+F 6 "A98038-ND" H 8200 6000 50  0001 C CNN "Digi-Key_PN"
+	1    8200 6000
+	-1   0    0    -1
 $EndComp
 $Comp
-L Connector_Generic:Conn_01x04 J?
+L Connector_Generic:Conn_01x04 J2
 U 1 1 5D619CD2
 P 9100 6000
-F 0 "J?" H 9179 5992 50  0000 L CNN
+F 0 "J2" H 9179 5992 50  0000 L CNN
 F 1 "JST-PH" H 9179 5901 50  0000 L CNN
 F 2 "Connector_JST:JST_PH_B4B-PH-K_1x04_P2.00mm_Vertical" H 9100 6000 50  0001 C CNN
@@
 	1    0    0    -1
 $EndComp
+Wire Wire Line
+	8400 5900 8900 5900
+Wire Wire Line
+	8400 6000 8900 6000
+Wire Wire Line
+	8400 6100 8900 6100
+Wire Wire Line
+	8400 6200 8900 6200
 $EndSCHEMATC

Commit message: Use right-angle JST-PH connector.
Parts:
- J2: footprint Connector_JST:JST_PH_B4B-PH-K_1x04_P2.00mm_Vertical -> Connector_JST:JST_PH_S4B-PH-K_1x04_P2.00mm_Horizontal; Description CONN HEADER VERT 4POS 2MM -> CONN HEADER R/A 4POS 2MM; Digi-Key_PN 455-1706-ND -> 455-1721-ND; MPN B4B-PH-K-S(LF)(SN) -> S4B-PH-K-S(LF)(SN)
Changed lines of the file:
@@
 EESchema Schematic File Version 4
+LIBS:SpeakerAdapter-cache
 EELAYER 26 0
 EELAYER END
@@
 F 0 "J2" H 9179 5992 50  0000 L CNN
 F 1 "JST-PH" H 9179 5901 50  0000 L CNN
-F 2 "Connector_JST:JST_PH_B4B-PH-K_1x04_P2.00mm_Vertical" H 9100 6000 50  0001 C CNN
+F 2 "Connector_JST:JST_PH_S4B-PH-K_1x04_P2.00mm_Horizontal" H 9100 6000 50  0001 C CNN
 F 3 "http://www.jst-mfg.com/product/pdf/eng/ePH.pdf" H 9100 6000 50  0001 C CNN
-F 4 "B4B-PH-K-S(LF)(SN)" H 9100 6000 50  0001 C CNN "MPN"
-F 5 "CONN HEADER VERT 4POS 2MM" H 9100 6000 50  0001 C CNN "Description"
-F 6 "455-1706-ND" H 9100 6000 50  0001 C CNN "Digi-Key_PN"
+F 4 "S4B-PH-K-S(LF)(SN)" H 9100 6000 50  0001 C CNN "MPN"
+F 5 "CONN HEADER R/A 4POS 2MM" H 9100 6000 50  0001 C CNN "Description"
+F 6 "455-1721-ND" H 9100 6000 50  0001 C CNN "Digi-Key_PN"
 	1    9100 6000
 	1    0    0    -1

Commit message: Use new terminal block footprint with no silk.
Parts:
- J1: footprint TerminalBlock_4Ucon:TerminalBlock_4Ucon_1x04_P3.50mm_Horizontal -> local:TerminalBlock_4Ucon_1x04_P3.50mm_Horizontal
Changed lines of the file:
@@
 F 0 "J1" H 8279 5992 50  0000 L CNN
 F 1 "Terminal Block" H 8279 5901 50  0000 L CNN
-F 2 "TerminalBlock_4Ucon:TerminalBlock_4Ucon_1x04_P3.50mm_Horizontal" H 8200 6000 50  0001 C CNN
+F 2 "local:TerminalBlock_4Ucon_1x04_P3.50mm_Horizontal" H 8200 6000 50  0001 C CNN
 F 3 "~" H 8200 6000 50  0001 C CNN
 F 4 "1776275-4" H 8200 6000 50  0001 C CNN "MPN"
